Commit message: Documentation pass to the family standard; remove dead hardware paths; IMU orientation filter
Docs, per the 4Cs and the wk-robotics conventions: AGENTS.md is the provider-neutral
onboarding (CLAUDE.md and GEMINI.md point at it); docs/ gains concept, architecture,
hardware, operations, decisions (DEC-01..19), open-questions (OQ-01..13), roadmap,
references and test-log, in the wk-devastator format. README is the human entry.
The old CLAUDE.md content and docs/ubuntu-hardware-setup.md are absorbed. No host
names remain in the public repo (mission.sh defaults to localhost).

Removed as superfluous or incoherent: the ultrasonic range-finder driver and the Pi
Camera node (hardware no longer fitted), the slam_toolbox launch/params/dependency
(RTAB-Map is the decided SLAM), the duplicate root config/ (unused params.json and a
second copy of the calibration), the vendor PDF, the URDF ultrasonic link, and
bring-up's robot.yaml (body_params.yaml in hexapod_controller is the single controller
config, matching the parameters the node declares).

Fixed: the controller subscribed to /imu/data with orientation while the driver
publishes /imu/data_raw without it, so IMU yaw fusion had never received data;
imu_filter_madgwick now bridges them (DEC-19, conventions unverified: OQ-13). The
controller no longer publishes during shutdown after the context is gone.
controller.launch.py exposes direct_hardware for standalone use. Package metadata
carries the real maintainer and accurate descriptions.

Verified: full stack restarted under systemd, 37 nodes, /imu/data carries a
quaternion, clean shutdown, buzzer pin still held by the guard.

Co-Authored-By: Claude Fable 5.1 <noreply@anthropic.com>
Claude-Session: https://claude.ai/code/session_01QRQzZ3McihxKEqMy7p7RgH

File: ros2_ws/src/hexapod_bringup/urdf/hexapod.urdf (robot description, URDF)
Before this commit: robot hexapod, 13 links, 12 joints
Links:
- removed link ultrasonic_link
Joints:
- removed joint ultrasonic_joint

Commit message: Sonar and head stack replaces the D435i (DEC-25, DEC-27, DEC-28)
Written on the robot 2026-09-19 as 343638f and never pushed; merged from the workstation
2026-09-21 (DEC-29, OQ-24). Renumbered on merge because main had assigned DEC-26 and OQ-19
first: the robot's DEC-26 is DEC-27, its DEC-27 is DEC-28, and its OQ-19..22 are OQ-20..23.
Conflicts resolved:
- decisions.md: the robot's DEC-25 is folded into main's DEC-25 as its implementation.
- open-questions.md: main's OQ-19 (mapping without depth) is marked resolved by it.
- docs: the robot's current-state text wins. Kept from main: DEC-26 in AGENTS.md, the
  Orin Nano destination, and the 2026-09-18 decision in concept.md's chronology.
- ubuntu-setup.sh: main's UTC step plus the robot's camera changes, renumbered 1-9.
ros2_ws is byte-identical to 343638f (tree c0aa89f), so the robot's running code is unchanged.

Co-Authored-By: Claude Opus 5 (1M context) <noreply@anthropic.com>
Claude-Session: https://claude.ai/code/session_01Kbp268oPe7jXWTMZrDC62k

File: ros2_ws/src/hexapod_bringup/urdf/hexapod.urdf (robot description, URDF)
Before this commit: robot hexapod, 12 links, 11 joints
Links:
- removed link camera_color_frame
- removed link camera_color_optical_frame
- removed link camera_depth_frame
- removed link camera_depth_optical_frame
- removed link camera_imu_optical_frame
- removed link laser_frame
- added link camera_optical_frame
- added link ultrasonic_link; visual box size=0.015 0.045 0.02
- link camera_link: geometry visual box size=0.01 0.025 0.024
Joints:
- removed joint camera_color_joint
- removed joint camera_color_optical_joint
- removed joint camera_depth_joint
- removed joint camera_depth_optical_joint
- removed joint camera_imu_joint
- removed joint laser_joint
- added joint camera_optical_joint: type fixed, parent camera_link, child camera_optical_frame, origin xyz=0 0 0 rpy=-1.5708 0 -1.5708
- added joint ultrasonic_joint: type fixed, parent head_tilt_link, child ultrasonic_link, origin xyz=0.03 0 0 rpy=0 0 0
- joint camera_joint: origin xyz=0.03 0 0.01 rpy=0 0 0 -> xyz=0.03 0 0.025 rpy=0 0 0

Commit message: Lidar: RPLIDAR C1 on /scan via sllidar_ros2 (pinned), laser_frame, standalone slam_toolbox launch
Co-Authored-By: Claude Opus 5.5 (1M context) <noreply@anthropic.com>
Claude-Session: https://claude.ai/code/session_01F6zLaYKCmA3dibVQ8pser5

File: ros2_ws/src/hexapod_bringup/urdf/hexapod.urdf (robot description, URDF)
Before this commit: robot hexapod, 8 links, 7 joints
Links:
- added link laser_frame
Joints:
- added joint laser_joint: type fixed, parent base_link, child laser_frame, origin xyz=0 0 0.16 rpy=0 0 0

Commit message: URDF: laser_frame yaw pi, from the bench test (boxes ahead at 180 deg, wall behind at 0, pole behind-left at -50)
Co-Authored-By: Claude Opus 5.5 (1M context) <noreply@anthropic.com>
Claude-Session: https://claude.ai/code/session_01F6zLaYKCmA3dibVQ8pser5

File: ros2_ws/src/hexapod_bringup/urdf/hexapod.urdf (robot description, URDF)
Before this commit: robot hexapod, 9 links, 8 joints
Joints:
- joint laser_joint: origin xyz=0 0 0.16 rpy=0 0 0 -> xyz=0 0 0.16 rpy=0 0 3.14159265

Commit message: URDF: laser_frame x +0.010 m, y 0 (owner-measured plan position)
Co-Authored-By: Claude Opus 5.5 (1M context) <noreply@anthropic.com>
Claude-Session: https://claude.ai/code/session_01F6zLaYKCmA3dibVQ8pser5

File: ros2_ws/src/hexapod_bringup/urdf/hexapod.urdf (robot description, URDF)
Before this commit: robot hexapod, 9 links, 8 joints
Joints:
- joint laser_joint: origin xyz=0 0 0.16 rpy=0 0 3.14159265 -> xyz=0.010 0 0.16 rpy=0 0 3.14159265
